File: coqui-dip.sch (EAGLE design)
At the start: 4 parts

Commit message: update
Parts:
- removed IC1: (no value), SparkFun-AnalogIC:556
- added C3: 0.01uF, rcl:C-EUC0805
- added C7: 0.1uF, rcl:C-EUC0805
- added IC2, IC3: LM555D, adafruit:LM555D
- added J1: AYZ0202, SparkFunNew:AYZ0202
- added JP1: (no value), SparkFun-Connectors:M04PTH
- added JP2: M10", SparkFun-Connectors:M10"
- added JP3, JP4: (no value), SparkFun-Connectors:M06SIP
- added R1, R2: M02PTH, SparkFun-Connectors:M02PTH
- C1: value (none) -> 0.1uF; device SparkFun-Capacitors:CAPPTH1 -> rcl:C-EUC0805
- C2: value (none) -> 0.01uF; device SparkFun-Capacitors:CAPPTH1 -> rcl:C-EUC0805
Connections:
- new net N$2: J1.1, J1.4
- new net VBAT: J1.2, J1.5
- new net VDD: J1.3, J1.6
Other:
- moved on the sheet: C1, C2
Changed lines of the file:
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@@
 </variantdefs>
 <classes>
-<class number="0" name="default" width="0" drill="0">
+<class number="0" name="default" width="0.254" drill="0">
+<clearance class="0" value="0.2032"/>
 </class>
 </classes>
 <parts>
-<part name="IC1" library="SparkFun-AnalogIC" deviceset="556" device=""/>
 <part name="GND4" library="supply1" deviceset="GND" device=""/>
 <part name="U$1" library="iPhoneSoftModem" deviceset="MJ-2135" device=""/>
-<part name="C1" library="SparkFun-Capacitors" deviceset="CAP" device="PTH1"/>
-<part name="C2" library="SparkFun-Capacitors" deviceset="CAP" device="PTH1"/>
+<part name="IC2" library="adafruit" deviceset="*555" device="D" technology="LM"/>
+<part name="IC3" library="adafruit" deviceset="*555" device="D" technology="LM"/>
+<part name="C7" library="rcl" deviceset="C-EU" device="C0805" value="0.1uF"/>
+<part name="R1" library="SparkFun-Connectors" deviceset="M02" device="PTH"/>
+<part name="R2" library="SparkFun-Connectors" deviceset="M02" device="PTH"/>
+<part name="C1" library="rcl" deviceset="C-EU" device="C0805" value="0.1uF"/>
+<part name="C2" library="rcl" deviceset="C-EU" device="C0805" value="0.01uF"/>
+<part name="C3" library="rcl" deviceset="C-EU" device="C0805" value="0.01uF"/>
+<part name="J1" library="SparkFunNew" deviceset="AYZ0202" device=""/>
+<part name="JP3" library="SparkFun-Connectors" deviceset="M06" device="SIP"/>
+<part name="JP4" library="SparkFun-Connectors" deviceset="M06" device="SIP"/>
+<part name="JP1" library="SparkFun-Connectors" deviceset="M04" device="PTH"/>
+<part name="JP2" library="SparkFun-Connectors" deviceset="M10" device="&quot;"/>
 </parts>
 <sheets>
@@
 </plain>
 <instances>
-<instance part="IC1" gate="G$1" x="38.1" y="58.42"/>
 <instance part="GND4" gate="1" x="0" y="88.9"/>
 <instance part="U$1" gate="G$1" x="-5.08" y="99.06"/>
-<instance part="C1" gate="G$1" x="35.56" y="91.44"/>
-<instance part="C2" gate="G$1" x="48.26" y="91.44"/>
+<instance part="IC2" gate="A" x="78.74" y="55.88"/>
+<instance part="IC3" gate="A" x="114.3" y="55.88"/>
+<instance part="C7" gate="G$1" x="80.01" y="90.17" smashed="yes" rot="R90">
+<attribute name="NAME" x="77.724" y="88.011" size="1.778" layer="95"/>
+<attribute name="VALUE" x="77.724" y="85.471" size="1.778" layer="96"/>
+</instance>
+<instance part="R1" gate="G$1" x="-33.02" y="63.5"/>
+<instance part="R2" gate="G$1" x="-33.02" y="45.72"/>
+<instance part="C1" gate="G$1" x="59.69" y="87.63" smashed="yes" rot="R90">
+<attribute name="NAME" x="57.404" y="85.471" size="1.778" layer="95"/>
+<attribute name="VALUE" x="57.404" y="82.931" size="1.778" layer="96"/>
+</instance>
+<instance part="C2" gate="G$1" x="52.07" y="97.79" smashed="yes" rot="R90">
+<attribute name="NAME" x="49.784" y="95.631" size="1.778" layer="95"/>
+<attribute name="VALUE" x="49.784" y="93.091" size="1.778" layer="96"/>
+</instance>
+<instance part="C3" gate="G$1" x="67.31" y="97.79" smashed="yes" rot="R90">
+<attribute name="NAME" x="65.024" y="95.631" size="1.778" layer="95"/>
+<attribute name="VALUE" x="65.024" y="93.091" size="1.778" layer="96"/>
+</instance>
+<instance part="J1" gate="G$1" x="27.94" y="66.04" smashed="yes">
+<attribute name="NAME" x="25.4" y="74.168" size="1.778" layer="95"/>
+</instance>
+<instance part="JP3" gate="G$1" x="86.36" y="106.68"/>
+<instance part="JP4" gate="G$1" x="104.14" y="106.68"/>
+<instance part="JP1" gate="G$1" x="53.34" y="63.5"/>
+<instance part="JP2" gate="G$1" x="134.62" y="99.06"/>
 </instances>
 <busses>
@@
 </segment>
 </net>
+<net name="VDD" class="0">
+<segment>
+<pinref part="J1" gate="G$1" pin="3"/>
+<pinref part="J1" gate="G$1" pin="6"/>
+<wire x1="33.02" y1="66.04" x2="33.02" y2="62.23" width="0.1524" layer="91"/>
+<wire x1="33.02" y1="62.23" x2="33.02" y2="58.42" width="0.1524" layer="91"/>
+<wire x1="33.02" y1="62.23" x2="36.83" y2="62.23" width="0.1524" layer="91"/>
+<junction x="33.02" y="62.23"/>
+</segment>
+</net>
+<net name="VBAT" class="0">
+<segment>
+<wire x1="20.32" y1="64.77" x2="22.86" y2="64.77" width="0.1524" layer="91"/>
+<pinref part="J1" gate="G$1" pin="2"/>
+<wire x1="22.86" y1="68.58" x2="22.86" y2="64.77" width="0.1524" layer="91"/>
+<pinref part="J1" gate="G$1" pin="5"/>
+<wire x1="22.86" y1="64.77" x2="22.86" y2="60.96" width="0.1524" layer="91"/>
+<junction x="22.86" y="64.77"/>
+</segment>
+</net>
+<net name="N$2" class="0">
+<segment>
+<pinref part="J1" gate="G$1" pin="1"/>
+<wire x1="33.02" y1="71.12" x2="34.29" y2="71.12" width="0.1524" layer="91"/>
+<wire x1="34.29" y1="71.12" x2="34.29" y2="63.5" width="0.1524" layer="91"/>
+<pinref part="J1" gate="G$1" pin="4"/>
+<wire x1="34.29" y1="63.5" x2="33.02" y2="63.5" width="0.1524" layer="91"/>
+</segment>
+</net>

Commit message: update
Parts:
- removed JP1: (no value), SparkFun-Connectors:M04PTH
- removed JP3, JP4: (no value), SparkFun-Connectors:M06SIP
- removed R1, R2: M02PTH, SparkFun-Connectors:M02PTH
- added BAT: CR1220, SparkFunNew:BATTERYBATTERY_12MM_SMT
- added C4, C5, C6, C8: 0.1uF, rcl:C-EUC0805
- added J2: AYZ0202, SparkFunNew:AYZ0202
- added JP5: M20, SparkFun-Connectors:M20
- added JP6: (no value), SparkFun-Connectors:M081X08
- JP2: value M10" -> (none); device SparkFun-Connectors:M10" -> SparkFun-Connectors:M081X08
Connections:
- new net GND1: BAT.-
- new net N$3: J2.1, J2.4
- new net VBAT1: J2.2, J2.5
- new net VDD1: J2.3, J2.6
Changed lines of the file:
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@@
 </variantdefs>
 <classes>
-<class number="0" name="default" width="0.254" drill="0">
+<class number="0" name="default" width="0.2032" drill="0.3302">
 <clearance class="0" value="0.2032"/>
 </class>
@@
 <part name="IC3" library="adafruit" deviceset="*555" device="D" technology="LM"/>
 <part name="C7" library="rcl" deviceset="C-EU" device="C0805" value="0.1uF"/>
-<part name="R1" library="SparkFun-Connectors" deviceset="M02" device="PTH"/>
-<part name="R2" library="SparkFun-Connectors" deviceset="M02" device="PTH"/>
 <part name="C1" library="rcl" deviceset="C-EU" device="C0805" value="0.1uF"/>
 <part name="C2" library="rcl" deviceset="C-EU" device="C0805" value="0.01uF"/>
 <part name="C3" library="rcl" deviceset="C-EU" device="C0805" value="0.01uF"/>
 <part name="J1" library="SparkFunNew" deviceset="AYZ0202" device=""/>
-<part name="JP3" library="SparkFun-Connectors" deviceset="M06" device="SIP"/>
-<part name="JP4" library="SparkFun-Connectors" deviceset="M06" device="SIP"/>
-<part name="JP1" library="SparkFun-Connectors" deviceset="M04" device="PTH"/>
-<part name="JP2" library="SparkFun-Connectors" deviceset="M10" device="&quot;"/>
+<part name="JP5" library="SparkFun-Connectors" deviceset="M20" device=""/>
+<part name="JP2" library="SparkFun-Connectors" deviceset="M08" device="1X08"/>
+<part name="JP6" library="SparkFun-Connectors" deviceset="M08" device="1X08"/>
+<part name="C4" library="rcl" deviceset="C-EU" device="C0805" value="0.1uF"/>
+<part name="C5" library="rcl" deviceset="C-EU" device="C0805" value="0.1uF"/>
+<part name="J2" library="SparkFunNew" deviceset="AYZ0202" device=""/>
+<part name="BAT" library="SparkFunNew" deviceset="BATTERY" device="BATTERY_12MM_SMT" value="CR1220"/>
+<part name="C6" library="rcl" deviceset="C-EU" device="C0805" value="0.1uF"/>
+<part name="C8" library="rcl" deviceset="C-EU" device="C0805" value="0.1uF"/>
 </parts>
 <sheets>
@@
 <attribute name="VALUE" x="77.724" y="85.471" size="1.778" layer="96"/>
 </instance>
-<instance part="R1" gate="G$1" x="-33.02" y="63.5"/>
-<instance part="R2" gate="G$1" x="-33.02" y="45.72"/>
 <instance part="C1" gate="G$1" x="59.69" y="87.63" smashed="yes" rot="R90">
 <attribute name="NAME" x="57.404" y="85.471" size="1.778" layer="95"/>
@@
 <attribute name="NAME" x="25.4" y="74.168" size="1.778" layer="95"/>
 </instance>
-<instance part="JP3" gate="G$1" x="86.36" y="106.68"/>
-<instance part="JP4" gate="G$1" x="104.14" y="106.68"/>
-<instance part="JP1" gate="G$1" x="53.34" y="63.5"/>
-<instance part="JP2" gate="G$1" x="134.62" y="99.06"/>
+<instance part="JP5" gate="G$1" x="7.62" y="35.56"/>
+<instance part="JP2" gate="G$1" x="40.64" y="30.48"/>
+<instance part="JP6" gate="G$1" x="55.88" y="30.48"/>
+<instance part="C4" gate="G$1" x="92.71" y="80.01" smashed="yes" rot="R90">
+<attribute name="NAME" x="90.424" y="77.851" size="1.778" layer="95"/>
+<attribute name="VALUE" x="90.424" y="75.311" size="1.778" layer="96"/>
+</instance>
+<instance part="C5" gate="G$1" x="72.39" y="77.47" smashed="yes" rot="R90">
+<attribute name="NAME" x="70.104" y="75.311" size="1.778" layer="95"/>
+<attribute name="VALUE" x="70.104" y="72.771" size="1.778" layer="96"/>
+</instance>
+<instance part="J2" gate="G$1" x="30.48" y="101.6" smashed="yes">
+<attribute name="NAME" x="27.94" y="109.728" size="1.778" layer="95"/>
+</instance>
+<instance part="BAT" gate="G$1" x="-24.13" y="60.452" smashed="yes" rot="R270">
+<attribute name="NAME" x="-19.05" y="60.452" size="1.778" layer="95"/>
+<attribute name="VALUE" x="-19.05" y="57.912" size="1.778" layer="96"/>
+</instance>
+<instance part="C6" gate="G$1" x="123.19" y="85.09" smashed="yes" rot="R90">
+<attribute name="NAME" x="120.904" y="82.931" size="1.778" layer="95"/>
+<attribute name="VALUE" x="120.904" y="80.391" size="1.778" layer="96"/>
+</instance>
+<instance part="C8" gate="G$1" x="102.87" y="82.55" smashed="yes" rot="R90">
+<attribute name="NAME" x="100.584" y="80.391" size="1.778" layer="95"/>
+<attribute name="VALUE" x="100.584" y="77.851" size="1.778" layer="96"/>
+</instance>
 </instances>
 <busses>
@@
 </segment>
 </net>
+<net name="VDD1" class="0">
+<segment>
+<pinref part="J2" gate="G$1" pin="3"/>
+<pinref part="J2" gate="G$1" pin="6"/>
+<wire x1="35.56" y1="101.6" x2="35.56" y2="97.79" width="0.1524" layer="91"/>
+<wire x1="35.56" y1="97.79" x2="35.56" y2="93.98" width="0.1524" layer="91"/>
+<wire x1="35.56" y1="97.79" x2="39.37" y2="97.79" width="0.1524" layer="91"/>
+<junction x="35.56" y="97.79"/>
+</segment>
+</net>
+<net name="VBAT1" class="0">
+<segment>
+<wire x1="22.86" y1="100.33" x2="25.4" y2="100.33" width="0.1524" layer="91"/>
+<pinref part="J2" gate="G$1" pin="2"/>
+<wire x1="25.4" y1="104.14" x2="25.4" y2="100.33" width="0.1524" layer="91"/>
+<pinref part="J2" gate="G$1" pin="5"/>
+<wire x1="25.4" y1="100.33" x2="25.4" y2="96.52" width="0.1524" layer="91"/>
+<junction x="25.4" y="100.33"/>
+</segment>
+</net>
+<net name="N$3" class="0">
+<segment>
+<pinref part="J2" gate="G$1" pin="1"/>
+<wire x1="35.56" y1="106.68" x2="36.83" y2="106.68" width="0.1524" layer="91"/>
+<wire x1="36.83" y1="106.68" x2="36.83" y2="99.06" width="0.1524" layer="91"/>
+<pinref part="J2" gate="G$1" pin="4"/>
+<wire x1="36.83" y1="99.06" x2="35.56" y2="99.06" width="0.1524" layer="91"/>
+</segment>
+</net>
+<net name="GND1" class="0">
+<segment>
+<wire x1="-24.13" y1="55.372" x2="-24.13" y2="48.26" width="0.1524" layer="91"/>
+<pinref part="BAT" gate="G$1" pin="-"/>
+</segment>
+</net>
