File: coqui-dip-body.sch (EAGLE design)
At the start: 14 parts, among them IC1 OPAMP-DUALU, IC2 LM555D, IC3 LM555D

Commit message: update
Parts:
- removed BAT: CR1220, SparkFunNew:BATTERYBATTERY_12MM_SMT
- removed JP5: M20, SparkFun-Connectors:M20
- added BAT1: LIR2032, SparkFunNew:BATTERYBATTCOM_20MM_PTH_SMT
- added CHG: 0805, led:LEDCHIPLED_0805
- added CN1: (no value), adafruit:JST_2PIN-SMT-RA
- added IC4: MCP73831, SparkFunNew:MCP73831
- added IC5: MCP1700-33, adafruit:MCP1700SOT89
- added J-FEMALE: MJ-2135, iPhoneSoftModem:MJ-2135
- added J1: AYZ0202, SparkFunNew:AYZ0202
- added JACK1: (no value), con-lstb:MA04-1
- added JP1: (no value), trrs-dwb:PINHD-1X4/90
- added JP2: (no value), pinhead:PINHD-1X18
- added R2, RV: M02PTH, SparkFun-Connectors:M02PTH
- added RB: 1, adafruit2013:R-US_R0805
- added RC, RC1: 4.7K, adafruit2013:R-US_R0805
- added X1: USBSMD, SparkFun:USBSMD
- U$1: value MJ-2135 -> BUZZER; device iPhoneSoftModem:MJ-2135 -> adafruit:BUZZER
Connections:
- removed net GND1: BAT.-
- new net N$12: RB.1, U$1.+
- new net N$2: J-FEMALE.2, JP1.1
- new net N$3: IC4.PROG, RC.2
- new net N$4: X1.GND
- new net N$5: CHG.C, IC4.STAT
- new net N$7: U$1.-, U$1.A-
- new net N$8: CHG.A, RC1.1
- new net VBAT: BAT1.+, CN1.2, IC4.VBAT, J1.2
- new net VBUS: IC4.VIN, RC1.2, X1.VBUS
- new net VCC: IC5.OUT
- new net VDD: IC5.IN, J1.3
- net GND: now also BAT1.-, CN1.1, IC4.VSS, IC5.GND, J-FEMALE.3, RC.1; no longer U$1.3
- net N$1: now also J-FEMALE.4; no longer U$1.4
- net N$6: now also J-FEMALE.1; no longer U$1.1
Other:
- moved on the sheet: R1
