File: coqui-dip-body.brd (EAGLE design)
At the start: 39 x 38.1 mm, 14 parts, among them IC1 OPAMP-DUALU, IC2 LM555D, IC3 LM555D

Commit message: yes.
Parts:
- moved BAT 8.52 mm to (7.62, 24.1), turned to 270 degrees
- moved JP5 5.08 mm to (0.00, 45.7)
- moved C1 2.54 mm to (6.35, 14.0)
- moved C2 2.54 mm to (29.2, 14.0)
- moved R1 2.54 mm to (20.3, 17.8)
- moved IC2 2.54 mm to (30.5, 7.62)
- moved IC3 2.54 mm to (7.62, 7.62), turned to 0 degrees
- moved CA 1.27 mm to (7.62, 1.27)
- moved CB 1.27 mm to (30.5, 1.27)
- turned IC1 to 90 degrees
Other:
- board size 39 x 38.1 mm -> 37.8 x 33 mm
Changed lines of the file:
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@@
 <board>
 <plain>
-<wire x1="0" y1="0" x2="39.04" y2="0" width="0" layer="20"/>
-<wire x1="39.04" y1="0" x2="39.04" y2="38.09" width="0" layer="20"/>
-<wire x1="39.04" y1="38.09" x2="0" y2="38.09" width="0" layer="20"/>
-<wire x1="0" y1="38.09" x2="0" y2="0" width="0" layer="20"/>
+<wire x1="0" y1="0" x2="37.77" y2="0" width="0" layer="20"/>
+<wire x1="37.77" y1="0" x2="37.77" y2="33.01" width="0" layer="20"/>
+<wire x1="37.77" y1="33.01" x2="0" y2="33.01" width="0" layer="20"/>
+<wire x1="0" y1="33.01" x2="0" y2="0" width="0" layer="20"/>
+<wire x1="36.83" y1="21.59" x2="21.59" y2="24.13" width="0" layer="20" curve="198.434949"/>
 </plain>
 <attributes>
@@
 <elements>
 <element name="U$1" library="iPhoneSoftModem" package="MJ-2135" value="MJ-2135" x="25.4" y="13.97" rot="R180"/>
-<element name="IC2" library="adafruit" package="SO08" value="LM555D" x="30.48" y="10.16" rot="R180"/>
-<element name="IC3" library="adafruit" package="SO08" value="LM555D" x="7.62" y="10.16" rot="R180"/>
-<element name="CA" library="rcl" package="C0805@1" value="0.01uF" x="7.62" y="2.54"/>
-<element name="CB" library="rcl" package="C0805@1" value="0.01uF" x="30.48" y="2.54"/>
-<element name="JP5" library="SparkFun-Connectors" package="1X20" value="M20" x="5.08" y="45.72"/>
-<element name="BAT" library="SparkFunNew" package="BATTCON_12MM_SMT" value="CR1220" x="15.24" y="27.94" rot="R180"/>
-<element name="IC1" library="SparkFun-AnalogIC" package="SO08" value="OPAMP-DUALU" x="29.21" y="24.13" rot="R270"/>
-<element name="C1" library="SparkFun-Connectors" package="1X02" value="M02PTH" x="6.35" y="16.51"/>
-<element name="C2" library="SparkFun-Connectors" package="1X02" value="M02PTH" x="29.21" y="16.51"/>
-<element name="R1" library="SparkFun-Connectors" package="1X02" value="M02PTH" x="20.32" y="15.24"/>
+<element name="IC2" library="adafruit" package="SO08" value="LM555D" x="30.48" y="7.62" rot="R180"/>
+<element name="IC3" library="adafruit" package="SO08" value="LM555D" x="7.62" y="7.62"/>
+<element name="CA" library="rcl" package="C0805@1" value="0.01uF" x="7.62" y="1.27"/>
+<element name="CB" library="rcl" package="C0805@1" value="0.01uF" x="30.48" y="1.27"/>
+<element name="JP5" library="SparkFun-Connectors" package="1X20" value="M20" x="0" y="45.72"/>
+<element name="BAT" library="SparkFunNew" package="BATTCON_12MM_SMT" value="CR1220" x="7.62" y="24.13" rot="R270"/>
+<element name="IC1" library="SparkFun-AnalogIC" package="SO08" value="OPAMP-DUALU" x="29.21" y="24.13" rot="R90"/>
+<element name="C1" library="SparkFun-Connectors" package="1X02" value="M02PTH" x="6.35" y="13.97"/>
+<element name="C2" library="SparkFun-Connectors" package="1X02" value="M02PTH" x="29.21" y="13.97"/>
+<element name="R1" library="SparkFun-Connectors" package="1X02" value="M02PTH" x="20.32" y="17.78"/>
 <element name="JACK" library="con-lstb" package="MA04-1" value="" x="13.97" y="6.35" rot="R90">
 <attribute name="OC_NEWARK" value="unknown" x="13.97" y="6.35" size="1.778" layer="27" rot="R90" display="off"/>
@@
 <contactref element="IC2" pad="1"/>
 <contactref element="IC3" pad="1"/>
-<wire x1="9.525" y1="13.2334" x2="32.385" y2="13.2334" width="0" layer="19" extent="1-1"/>
-<wire x1="19.1" y1="13.47" x2="9.525" y2="13.2334" width="0" layer="19" extent="1-1"/>
+<wire x1="5.715" y1="4.5466" x2="32.385" y2="10.6934" width="0" layer="19" extent="1-1"/>
+<wire x1="19.1" y1="13.47" x2="5.715" y2="4.5466" width="0" layer="19" extent="1-1"/>
 </signal>
 <signal name="N$6">
@@
 <contactref element="IC3" pad="8"/>
 <contactref element="IC1" pad="8"/>
-<wire x1="9.525" y1="7.0866" x2="32.385" y2="7.0866" width="0" layer="19" extent="1-1"/>
-<wire x1="31.8262" y1="26.035" x2="9.525" y2="7.0866" width="0" layer="19" extent="1-1"/>
+<wire x1="5.715" y1="10.6934" x2="32.385" y2="4.5466" width="0" layer="19" extent="1-1"/>
+<wire x1="26.5938" y1="22.225" x2="5.715" y2="10.6934" width="0" layer="19" extent="1-1"/>
 </signal>
 <signal name="+">

Commit message: update
Parts:
- removed BAT: CR1220, SparkFunNew:BATTCON_12MM_SMT
- removed JP5: M20, SparkFun-Connectors:1X20
- added BAT1: LIR2032, SparkFunNew:BATTCOM_20MM_PTH_SMT
- added CHG: 0805, led:CHIPLED_0805
- added CN1: (no value), adafruit:JST-PH-2-SMT-RA
- added IC4: MCP73831, SparkFunNew:SOT23-5
- added IC5: MCP1700-33, adafruit:SOT89
- added J-FEMALE: MJ-2135, iPhoneSoftModem:MJ-2135
- added J1: AYZ0202, SparkFunNew:AYZ0202
- added JACK1: (no value), con-lstb:MA04-1
- added JP1: (no value), trrs-dwb:1X04/90
- added JP2: (no value), pinhead:1X18
- added R2, RV: M02PTH, SparkFun-Connectors:1X02
- added RB: 1, adafruit2013:R0805
- added RC, RC1: 4.7K, adafruit2013:R0805
- added X1: USBSMD, SparkFun:USB-MINIB
- U$1: value MJ-2135 -> BUZZER; device iPhoneSoftModem:MJ-2135 -> adafruit:SMT-8585-BUZZER
- moved U$1 26.3 mm to (5.08, 30.7), turned to 0 degrees
- moved R1 24.0 mm to (7.62, 38.1)
- moved C2 14.2 mm to (43.4, 13.7), turned to 180 degrees
- moved IC2 11.7 mm to (42.2, 7.11)
- moved CB 11.7 mm to (42.2, 1.27), turned to 180 degrees
- moved JACK 9.25 mm to (22.6, 9.65), turned to 270 degrees
- moved SV2 7.62 mm to (8.89, 7.62)
- moved IC1 5.62 mm to (31.0, 18.8)
- moved CA 4.58 mm to (3.05, 1.52), turned to 180 degrees
- moved IC3 4.33 mm to (3.30, 7.37)
- moved C1 1.85 mm to (4.57, 14.5), turned to 180 degrees
Connections:
- removed net +: BAT.P$2
- removed net GND1: BAT.P$1
- new net N$12: RB.1, U$1.+
- new net N$2: J-FEMALE.2, JP1.1
- new net N$3: IC4.5, RC.2
- new net N$4: X1.GND
- new net N$5: CHG.C, IC4.1
- new net N$7: U$1.-, U$1.A-
- new net N$8: CHG.A, RC1.1
- new net VBAT: BAT1.P$2, CN1.1, IC4.3, J1.2
- new net VBUS: IC4.4, RC1.2, X1.VBUS
- new net VCC: IC5.3
- new net VDD: IC5.2, J1.1
- net GND: now also BAT1.P$1, CN1.2, IC4.2, IC5.1, J-FEMALE.3, RC.1; no longer U$1.3
- net N$1: now also J-FEMALE.4; no longer U$1.4
- net N$6: now also J-FEMALE.1; no longer U$1.1
Other:
- board size 37.8 x 33 mm -> 45.4 x 42.2 mm

Commit message: update
Parts:
- moved IC5 27.2 mm to (42.4, 38.1)
- moved R1 3.39 mm to (10.9, 38.9)
- moved RB 1.55 mm to (12.7, 35.6)
- moved R2 1.44 mm to (34.8, 38.9)
- moved RC1 0.57 mm to (20.8, 17.0)
Other:
- board size 45.4 x 42.2 mm -> 45.4 x 41.1 mm
Changed lines of the file:
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@@
 <plain>
 <wire x1="0" y1="0" x2="45.39" y2="0" width="0" layer="20"/>
-<wire x1="45.39" y1="0" x2="45.39" y2="42.154" width="0" layer="20"/>
-<wire x1="45.39" y1="42.154" x2="0" y2="42.154" width="0" layer="20"/>
-<wire x1="0" y1="42.154" x2="0" y2="0" width="0" layer="20"/>
+<wire x1="45.39" y1="0" x2="45.39" y2="41.138" width="0" layer="20"/>
+<wire x1="45.39" y1="41.138" x2="0" y2="41.138" width="0" layer="20"/>
+<wire x1="0" y1="41.138" x2="0" y2="0" width="0" layer="20"/>
 </plain>
 <attributes>
@@
 <element name="CN1" library="adafruit" package="JST-PH-2-SMT-RA" value="" x="3.81" y="21.082" rot="R90"/>
 <element name="J1" library="SparkFunNew" package="AYZ0202" value="AYZ0202" x="40.894" y="31.496" rot="R180"/>
-<element name="IC5" library="adafruit" package="SOT89" value="MCP1700-33" x="15.24" y="37.846" rot="R180"/>
+<element name="IC5" library="adafruit" package="SOT89" value="MCP1700-33" x="42.418" y="38.1" rot="R180"/>
 <element name="BAT1" library="SparkFunNew" package="BATTCOM_20MM_PTH_SMT" value="LIR2032" x="29.718" y="36.83" rot="R225"/>
 <element name="JP2" library="pinhead" package="1X18" value="" x="22.352" y="64.516"/>
@@
 </element>
 <element name="U$1" library="adafruit" package="SMT-8585-BUZZER" value="BUZZER" x="5.08" y="30.734"/>
-<element name="RB" library="adafruit2013" package="R0805" value="1" x="12.446" y="34.036" rot="R180"/>
-<element name="R1" library="SparkFun-Connectors" package="1X02" value="M02PTH" x="7.62" y="38.1"/>
-<element name="R2" library="SparkFun-Connectors" package="1X02" value="M02PTH" x="35.814" y="37.846"/>
-<element name="RC1" library="adafruit2013" package="R0805" value="4.7K" x="20.32" y="17.272"/>
+<element name="RB" library="adafruit2013" package="R0805" value="1" x="12.7" y="35.56" rot="R180"/>
+<element name="R1" library="SparkFun-Connectors" package="1X02" value="M02PTH" x="10.922" y="38.862"/>
+<element name="R2" library="SparkFun-Connectors" package="1X02" value="M02PTH" x="34.798" y="38.862"/>
+<element name="RC1" library="adafruit2013" package="R0805" value="4.7K" x="20.828" y="17.018"/>
 </elements>
 <signals>
@@
 <wire x1="29.718" y1="36.83" x2="35.56" y2="32.528" width="0" layer="19" extent="1-1"/>
 <wire x1="33.5581" y1="23.622" x2="35.56" y2="32.528" width="0" layer="19" extent="1-1"/>
-<wire x1="16.74" y1="39.646" x2="29.718" y2="36.83" width="0" layer="19" extent="1-1"/>
+<wire x1="43.918" y1="39.9" x2="29.718" y2="36.83" width="0" layer="19" extent="1-1"/>
 <wire x1="44.069" y1="10.1854" x2="33.5581" y2="23.622" width="0" layer="19" extent="1-1"/>
-<wire x1="7.51" y1="20.082" x2="16.74" y2="39.646" width="0" layer="19" extent="1-1"/>
+<wire x1="7.51" y1="20.082" x2="43.918" y2="39.9" width="0" layer="19" extent="1-1"/>
 <wire x1="13.004" y1="13.978" x2="7.51" y2="20.082" width="0" layer="19" extent="1-1"/>
 <wire x1="1.397" y1="4.2926" x2="13.004" y2="13.978" width="0" layer="19" extent="1-1"/>
@@
 <contactref element="RC1" pad="2"/>
 <wire x1="30.9579" y1="24.572" x2="37.378" y2="20.244" width="0" layer="19" extent="1-1"/>
-<wire x1="21.32" y1="17.272" x2="37.378" y2="20.244" width="0" layer="19" extent="1-1"/>
+<wire x1="21.828" y1="17.018" x2="37.378" y2="20.244" width="0" layer="19" extent="1-1"/>
 </signal>
 <signal name="VDD">
 <contactref element="J1" pad="1"/>
 <contactref element="IC5" pad="2"/>
-<wire x1="15.24" y1="39.646" x2="43.394" y2="28.671" width="0" layer="19" extent="1-1"/>
+<wire x1="42.418" y1="39.9" x2="43.394" y2="28.671" width="0" layer="19" extent="1-1"/>
 </signal>
 <signal name="N$5">
@@
 <contactref element="RB" pad="1"/>
 <contactref element="U$1" pad="+"/>
-<wire x1="1.58" y1="27.234" x2="13.446" y2="34.036" width="0" layer="19" extent="1-1"/>
+<wire x1="1.58" y1="27.234" x2="13.7" y2="35.56" width="0" layer="19" extent="1-1"/>
 </signal>
 <signal name="N$8">
 <contactref element="CHG" pad="A"/>
 <contactref element="RC1" pad="1"/>
-<wire x1="11.142" y1="17.018" x2="19.32" y2="17.272" width="0" layer="19" extent="1-1"/>
+<wire x1="11.142" y1="17.018" x2="19.828" y2="17.018" width="0" layer="19" extent="1-1"/>
 </signal>
 </signals>
