File: coqui-dip-simple.brd (EAGLE design)
At the start: 47.5 x 47.5 mm, 34 parts, among them IC1 OPAMP-DUALU, IC2 LM555D, IC3 LM555D, IC4 MCP73831, IC5 MCP1700-33, J1 AYZ0202, X1 USBSMD

Commit message: update
Parts:
- removed CA: 0.01uF, rcl:C0805@1
- removed CN1: (no value), adafruit:JST-PH-2-SMT-RA
- removed IC1: OPAMP-DUALU, SparkFun-AnalogIC:SO08
- removed IC2: LM555D, adafruit:SO08
- removed IC5: MCP1700-33, adafruit:SOT89
- removed MIC, R1, R2: M02PTH, SparkFun-Connectors:1X02
- removed RF, RS1, RS2: 1, adafruit2013:R0805
- removed SV1, SV2: (no value), con-lstb:MA06-1
- added BATT: (no value), adafruit:JST-PH-2-SMT-RA
- added CAN: 0.01uF, rcl:C0805@1
- added ICA, ICB: LM555D, adafruit:SO08
- added JP3, JP4: (no value), pinhead:1X04
- added RA: M02PTH, SparkFun-Connectors:1X02
- added RZ: 1, adafruit2013:R0805
- BZ: value M02PTH -> (none); device SparkFun-Connectors:1X02 -> pinhead:1X01
- IC3: value LM555D -> MCP73831; device adafruit:SO08 -> SparkFunNew:SOT23-5
- IC4: value MCP73831 -> MCP1700-33; device SparkFunNew:SOT23-5 -> adafruit:SOT89
- RB: value 1 -> M02PTH; device adafruit2013:R0805 -> SparkFun-Connectors:1X02
- moved RB 24.0 mm to (36.2, 45.0), turned to 324 degrees
- moved CHG 21.0 mm to (34.2, 19.6), turned to 180 degrees
- moved IC3 18.9 mm to (16.9, 19.3), turned to 180 degrees
- moved JP2 17.9 mm to (25.7, 50.2), flipped to the bottom
- moved RC 15.4 mm to (27.9, 19.7), turned to 270 degrees
- moved RC1 12.0 mm to (31.0, 19.6), turned to 90 degrees
- moved IC4 8.90 mm to (23.6, 19.4), turned to 180 degrees
- moved PWR 3.32 mm to (45.3, 32.3), turned to 270 degrees
- moved U$1 1.83 mm to (7.37, 35.1)
- moved J1 1.70 mm to (39.4, 36.6), turned to 90 degrees
- moved BZ 1.44 mm to (5.84, 28.2)
- moved JP1 1.14 mm to (31.0, 8.38)
- moved CB 0.54 mm to (43.3, 1.65)
- moved BAT1 0.52 mm to (30.5, 40.8)
- moved JACK 0.40 mm to (22.7, 9.78)
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Connections:
- removed net V-: IC1.4
- net GND: now also BATT.2, IC3.2, IC4.1, ICA.1, ICB.1, U$1.-, U$1.A-; no longer CN1.2, IC2.1, IC3.1, IC4.2, IC5.1
- net N$12: now also RZ.1; no longer RB.1
- net N$3: now also IC3.5; no longer IC4.5
- net N$5: now also IC3.1; no longer IC4.1
- net N$7: now also BZ.1, RZ.2; no longer U$1.-, U$1.A-
- net V+: now also ICA.8, ICB.8; no longer IC1.8, IC2.8, IC3.8
- net VBAT: now also BATT.1, IC3.3; no longer CN1.1, IC4.3
- net VBUS: now also IC3.4; no longer IC4.4
- net VCC: now also IC4.3; no longer IC5.3
- net VDD: now also IC4.2; no longer IC5.2
Other:
- board size 47.5 x 47.5 mm -> 48 x 13 mm
- board text added: "+"
- board text added: "1"
- board text added: "2"
- board text added: "3"
- board text added: "4"
- board text added: "555A"
- board text added: "555B"
- board text added: "C"
- board text added: "COQUI V1.0"
- board text added: "G"
- board text added: "IC3"
- board text added: "IC4"
- board text added: "O"
- board text added: "ON"
- board text added: "P"

Commit message: update
Parts:
- removed C2, RV: M02PTH, SparkFun-Connectors:1X02
- removed JACK, JACK1: (no value), con-lstb:MA04-1
- removed RC1: 4.7K, adafruit2013:R0805
- removed RZ: 1, adafruit2013:R0805
- added CAA, CBA, CBN: 0.01uF, rcl:C0805
- added JP5, JP6: (no value), pinhead:1X05
- added RN1: (no value), resistor-dil:EXB38V
- added RV1, RV2: 22K, adafruit2013:R0805
- CAN: device rcl:C0805@1 -> rcl:C0805
- CB: value 0.01uF -> M02PTH; device rcl:C0805@1 -> SparkFun-Connectors:1X02
- RC: value 4.7K -> 22K
- moved JP4 13.6 mm to (22.7, 6.22)
- moved CB 12.2 mm to (45.0, 13.7)
- moved JP3 7.92 mm to (29.2, 6.22)
- moved IC4 6.11 mm to (17.5, 19.1)
- moved IC3 6.03 mm to (10.9, 18.4)
- moved RC 5.03 mm to (23.0, 20.6), turned to 90 degrees
- moved JP2 3.27 mm to (24.9, 53.3)
- moved CHG 2.32 mm to (34.5, 17.3), turned to 0 degrees
- moved BZ 1.85 mm to (7.62, 28.7)
- moved JP1 1.40 mm to (30.9, 6.99)
- moved BATT 0.77 mm to (2.79, 22.1)
- moved X1 0.57 mm to (40.1, 22.6)
- moved PWR 0.52 mm to (45.2, 32.8)
- moved J1 0.25 mm to (39.4, 36.8)
- renumbered C1 to CA
Connections:
- removed net V+: ICA.8, ICB.8
- new net AOUT: ICB.3, JP5.5, RA.2, RN1.3, RV1.2
- new net BOUT: JP6.5, RB.2, RN1.4, RV2.2
- new net N$10: CAA.2, RV1.1
- new net N$11: CA.2, ICB.2, ICB.6, RA.1
- new net N$13: CBA.2, RV2.1
- new net N$14: CAN.2, ICB.5
- new net N$15: CBN.2, ICA.5
- new net N$16: CB.2, ICA.2, ICA.6, RB.1
- new net N$17: CBA.1, JP6.4
- new net N$18: JP1.1, JP3.1
- new net N$19: JP1.2, JP3.2
- new net N$20: JP1.3, JP3.3
- new net N$21: JP1.4, JP3.4
- new net N$9: CAA.1, JP5.4
- new net VAIN: ICB.4, ICB.8, JP5.3
- new net VBIN: ICA.4, ICA.8, JP6.3
- net GND: now also CA.1, CAN.1, CB.1, CBN.1, JP5.1, JP6.1, PWR.2, RN1.5, RN1.6, X1.GND; no longer J-FEMALE.3
- net N$1: now also J-FEMALE.1, JP4.1; no longer J-FEMALE.4
- net N$12: now also RN1.2; no longer RZ.1
- net N$2: now also JP4.2; no longer JP1.1
- net N$4: now also J-FEMALE.3, JP4.3; no longer X1.GND
- net N$6: now also J-FEMALE.4, JP4.4; no longer J-FEMALE.1
- net N$7: now also RN1.7; no longer RZ.2
- net N$8: now also RN1.1; no longer RC1.1
- net VBUS: now also RN1.8; no longer RC1.2
- net VCC: now also JP5.2, JP6.2
- net VDD: now also PWR.1
Other:
- board size 48 x 13 mm -> 48.1 x 49.3 mm
- board text added: "-"

Commit message: update
Parts:
- removed JP2: (no value), pinhead:1X18
- moved RN1 3.78 mm to (32.9, 28.3)
- moved RV1 0.97 mm to (22.2, 15.9)
- moved BZ 0.80 mm to (6.86, 28.4)
- moved CAN 0.74 mm to (2.54, 2.16)
- moved CBN 0.72 mm to (43.8, 2.16)
- moved CBA 0.63 mm to (31.9, 20.3)
- moved CAA 0.57 mm to (27.6, 20.3)
- moved RV2 0.57 mm to (29.6, 15.7)
- moved ICB 0.54 mm to (43.9, 7.87)
- moved RC 0.51 mm to (23.5, 20.6)
- moved CB 0.40 mm to (45.1, 14.1)
- moved IC3 0.38 mm to (10.9, 18.8)
- moved J1 0.18 mm to (39.5, 36.7), turned to 270 degrees
- moved ICA 0.13 mm to (2.29, 7.87)
Routing:
- net GND: track 0.00 -> 205.5 mm, vias 0 -> 1
- net AOUT: track 0.00 -> 106.6 mm, vias 0 -> 4
- net N$16: track 0.00 -> 105.1 mm, vias 0 -> 2
- net N$11: track 0.00 -> 89.6 mm, vias 0 -> 1
- net N$14: track 0.00 -> 56.3 mm, vias 0 -> 2
- net VCC: track 0.00 -> 51.6 mm
- net VBAT: track 0.00 -> 50.7 mm, vias 0 -> 3
- net BOUT: track 0.00 -> 49.6 mm, vias 0 -> 2
- net VDD: track 0.00 -> 48.1 mm, vias 0 -> 2
- net VAIN: track 0.00 -> 47.5 mm, vias 0 -> 1
- net VBIN: track 0.00 -> 47.0 mm, vias 0 -> 2
- net N$15: track 0.00 -> 44.8 mm, vias 0 -> 2
- net VBUS: track 0.00 -> 35.6 mm, vias 0 -> 3
- net N$12: track 0.00 -> 34.4 mm
- net N$7: track 0.00 -> 29.0 mm, vias 0 -> 3
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Other:
- board text added: "A"

Commit message: update
Routing:
- net VCC: track 51.6 -> 54.5 mm
Other:
- board text added: "http://publiclab.org/wiki/coqui"
Changed lines of the file:
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@@
 <layer number="17" name="Pads" color="2" fill="1" visible="yes" active="yes"/>
 <layer number="18" name="Vias" color="2" fill="1" visible="yes" active="yes"/>
-<layer number="19" name="Unrouted" color="6" fill="1" visible="no" active="yes"/>
+<layer number="19" name="Unrouted" color="6" fill="1" visible="yes" active="yes"/>
 <layer number="20" name="Dimension" color="15" fill="1" visible="yes" active="yes"/>
 <layer number="21" name="tPlace" color="7" fill="1" visible="yes" active="yes"/>
@@
 <rectangle x1="27.559" y1="11.43" x2="27.686" y2="13.081" layer="21"/>
 <rectangle x1="24.511" y1="11.43" x2="27.686" y2="11.557" layer="21"/>
-<text x="5.842" y="8.382" size="1.27" layer="21">A</text>
-<text x="5.969" y="6.096" size="1.27" layer="21">P</text>
-<text x="5.969" y="3.429" size="1.27" layer="21">+</text>
-<text x="5.842" y="1.016" size="1.27" layer="21">G</text>
+<text x="6.223" y="8.255" size="1.27" layer="21">A</text>
+<text x="6.35" y="5.461" size="1.27" layer="21">P</text>
+<text x="6.35" y="3.048" size="1.27" layer="21">+</text>
+<text x="6.35" y="0.635" size="1.27" layer="21">G</text>
 <text x="39.116" y="8.382" size="1.27" layer="21">A</text>
 <text x="39.243" y="5.842" size="1.27" layer="21">P</text>
-<text x="39.37" y="3.556" size="1.27" layer="21">+</text>
-<text x="39.116" y="0.889" size="1.27" layer="21">G</text>
+<text x="39.243" y="3.302" size="1.27" layer="21">+</text>
+<text x="39.243" y="0.381" size="1.27" layer="21">G</text>
 <text x="5.588" y="13.208" size="1.27" layer="21">C</text>
 <text x="39.37" y="13.462" size="1.27" layer="21">C</text>
 <text x="7.366" y="15.748" size="1.27" layer="21" rot="R315">555A</text>
 <text x="35.687" y="13.081" size="1.27" layer="21" rot="R45">555B</text>
-<text x="14.097" y="37.084" size="1.6764" layer="21" rot="R45">COQUI V1.0</text>
+<text x="13.843" y="36.322" size="1.6764" layer="21" rot="R45">COQUI V1.0</text>
 <text x="42.418" y="32.131" size="1.27" layer="21">+</text>
 <text x="42.545" y="29.718" size="1.27" layer="21">-</text>
 <text x="45.085" y="36.703" size="1.27" layer="21" rot="R90">ON</text>
-<text x="13.589" y="22.479" size="1.27" layer="21" rot="R180">IC3</text>
+<text x="14.097" y="22.733" size="1.27" layer="21" rot="R180">IC3</text>
 <text x="13.589" y="19.177" size="1.27" layer="21" rot="R270">IC4</text>
 <rectangle x1="-0.254" y1="16.129" x2="6.858" y2="16.383" layer="21"/>
@@
 <wire x1="4.572" y1="42.418" x2="4.826" y2="42.418" width="0" layer="20"/>
 <wire x1="47.117" y1="36.195" x2="47.117" y2="1.143" width="0" layer="20"/>
-<text x="5.842" y="10.795" size="1.27" layer="21">O</text>
+<text x="6.223" y="10.541" size="1.27" layer="21">O</text>
 <text x="39.37" y="10.795" size="1.27" layer="21">O</text>
+<text x="0.127" y="37.719" size="1.6764" layer="22" rot="MR180">http://publiclab.org/wiki/coqui</text>
 </plain>
 <attributes>
@@
 </element>
 <element name="CHG" library="led" package="CHIPLED_0805" value="0805" x="34.544" y="17.272" smashed="yes">
-<attribute name="NAME" x="35.433" y="22.098" size="1.27" layer="25" rot="R225"/>
+<attribute name="NAME" x="35.306" y="22.225" size="1.27" layer="25" rot="R225"/>
 <attribute name="VALUE" x="37.084" y="16.002" size="1.27" layer="27" rot="R90"/>
 </element>
@@
 <wire x1="11.2014" y1="18.1737" x2="11.5443" y2="18.5166" width="0.254" layer="1"/>
 <wire x1="11.2014" y1="11.0871" x2="11.2014" y2="18.1737" width="0.254" layer="1"/>
-<wire x1="13.9446" y1="8.3439" x2="11.2014" y2="11.0871" width="0.254" layer="1"/>
-<wire x1="13.9446" y1="5.715" x2="13.9446" y2="8.3439" width="0.254" layer="1"/>
+<wire x1="16.1036" y1="7.7089" x2="14.605" y2="9.271" width="0.254" layer="1"/>
+<wire x1="14.605" y1="9.271" x2="12.954" y2="11.0871" width="0.254" layer="1"/>
+<wire x1="12.954" y1="11.0871" x2="11.2014" y2="11.0871" width="0.254" layer="1"/>
+<wire x1="13.9446" y1="5.715" x2="16.1036" y2="7.7089" width="0.254" layer="1"/>
 <wire x1="12.0015" y1="3.7719" x2="13.20165" y2="4.97205" width="0.254" layer="1"/>
 <wire x1="13.20165" y1="4.97205" x2="13.9446" y2="5.715" width="0.254" layer="1"/>
@@
 <wire x1="4.6863" y1="3.429" x2="2.8575" y2="3.429" width="0.254" layer="1"/>
 <wire x1="7.2009" y1="5.9436" x2="4.6863" y2="3.429" width="0.254" layer="1"/>
-<wire x1="7.2009" y1="7.8867" x2="7.2009" y2="5.9436" width="0.254" layer="1"/>
-<wire x1="7.2009" y1="11.5443" x2="7.2009" y2="7.8867" width="0.254" layer="16"/>
+<wire x1="7.2009" y1="7.5057" x2="7.2009" y2="5.9436" width="0.254" layer="1"/>
+<wire x1="7.2009" y1="11.5443" x2="7.2009" y2="7.5057" width="0.254" layer="16"/>
 <wire x1="12.573" y1="16.9164" x2="7.2009" y2="11.5443" width="0.254" layer="16"/>
 <wire x1="29.3751" y1="16.9164" x2="12.573" y2="16.9164" width="0.254" layer="16"/>
@@
 <wire x1="1.6002" y1="2.1717" x2="1.59" y2="2.159" width="0.254" layer="1"/>
 <wire x1="42.0624" y1="4.8006" x2="42.037" y2="4.8006" width="0.254" layer="1"/>
-<via x="7.2009" y="7.8867" extent="1-16" drill="0.6096"/>
+<via x="7.2009" y="7.5057" extent="1-16" drill="0.6096"/>
 <via x="42.291" y="6.6294" extent="1-16" drill="0.6096"/>
 </signal>
@@
 <wire x1="18.8595" y1="12.2301" x2="19.8882" y2="12.2301" width="0.254" layer="16"/>
 <wire x1="16.6878" y1="10.0584" x2="18.8595" y2="12.2301" width="0.254" layer="16"/>
-<wire x1="10.9728" y1="10.0584" x2="16.6878" y2="10.0584" width="0.254" layer="16"/>
-<wire x1="8.1153" y1="10.0584" x2="10.9728" y2="10.0584" width="0.254" layer="1"/>
+<wire x1="11.6078" y1="10.0584" x2="16.6878" y2="10.0584" width="0.254" layer="16"/>
+<wire x1="8.1153" y1="10.0584" x2="11.6078" y2="10.0584" width="0.254" layer="1"/>
 <wire x1="4.1148" y1="6.0579" x2="8.1153" y2="10.0584" width="0.254" layer="1"/>
 <wire x1="37.1475" y1="6.4008" x2="37.211" y2="6.35" width="0.254" layer="1"/>
 <wire x1="4.1148" y1="6.0579" x2="4.1148" y2="5.9436" width="0.254" layer="1"/>
 <via x="19.8882" y="12.2301" extent="1-16" drill="0.6096"/>
-<via x="10.9728" y="10.0584" extent="1-16" drill="0.6096"/>
+<via x="11.6078" y="10.0584" extent="1-16" drill="0.6096"/>
 </signal>
 <signal name="N$17">
