File: coqui-dip-simple.sch (EAGLE design)
At the start: 34 parts, among them IC1 OPAMP-DUALU, IC2 LM555D, IC3 LM555D, IC4 MCP73831, IC5 MCP1700-33, J1 AYZ0202, X1 USBSMD

Commit message: update
Parts:
- removed IC1: OPAMP-DUALU, SparkFun-AnalogIC:OPAMP-DUALU
- removed IC5: MCP1700-33, adafruit:MCP1700SOT89
- removed MIC, R2: M02PTH, SparkFun-Connectors:M02PTH
- removed RF, RS1, RS2: 1, adafruit2013:R-US_R0805
- removed SV1, SV2: (no value), con-lstb:MA06-1
- added ICA: LM555D, adafruit:LM555D
- added JP3, JP4: (no value), pinhead:PINHD-1X4
- added RZ: 1, adafruit2013:R-US_R0805
- BZ: value M02PTH -> (none); device SparkFun-Connectors:M02PTH -> pinhead:PINHD-1X1
- IC3: value LM555D -> MCP73831; device adafruit:LM555D -> SparkFunNew:MCP73831
- IC4: value MCP73831 -> MCP1700-33; device SparkFunNew:MCP73831 -> adafruit:MCP1700SOT89
- RB: value 1 -> M02PTH; device adafruit2013:R-US_R0805 -> SparkFun-Connectors:M02PTH
- renumbered CA to CAN, CN1 to BATT, IC2 to ICB, R1 to RA
Connections:
- net GND: now also IC3.VSS, IC4.GND, U$1.-, U$1.A-; no longer IC4.VSS, IC5.GND
- net N$12: now also RZ.1; no longer RB.1
- net N$3: now also IC3.PROG; no longer IC4.PROG
- net N$5: now also IC3.STAT; no longer IC4.STAT
- net N$7: now also BZ.1, RZ.2; no longer U$1.-, U$1.A-
- net VBAT: now also IC3.VBAT; no longer IC4.VBAT
- net VBUS: now also IC3.VIN; no longer IC4.VIN
- net VCC: now also IC4.OUT; no longer IC5.OUT
- net VDD: now also IC4.IN; no longer IC5.IN

Commit message: update
Parts:
- removed C1, C2, RV: M02PTH, SparkFun-Connectors:M02PTH
- removed JACK, JACK1: (no value), con-lstb:MA04-1
- removed RC1: 4.7K, adafruit2013:R-US_R0805
- removed RZ: 1, adafruit2013:R-US_R0805
- added CA: M02PTH, SparkFun-Connectors:M02PTH
- added CAA, CBA, CBN: 0.01uF, rcl:C-EUC0805
- added JP5, JP6: (no value), pinhead:PINHD-1X5
- added RN1: (no value), resistor-dil:4R-NEXB38V
- added RV1, RV2: 22K, adafruit2013:R-US_R0805
- CB: value 0.01uF -> M02PTH; device rcl:C-EUC0805 -> SparkFun-Connectors:M02PTH
- RC: value 4.7K -> 22K
Connections:
- new net AOUT: ICB.Q, JP5.5, RA.2, RN1C.1, RV1.2
- new net BOUT: JP6.5, RB.2, RN1D.1, RV2.2
- new net N$10: CAA.2, RV1.1
- new net N$11: CA.2, ICB.THR, ICB.TR, RA.1
- new net N$13: CBA.2, RV2.1
- new net N$14: CAN.2, ICB.CV
- new net N$15: CBN.2, ICA.CV
- new net N$16: CB.2, ICA.THR, ICA.TR, RB.1
- new net N$17: CBA.1, JP6.4
- new net N$18: JP1.1, JP3.1
- new net N$19: JP1.2, JP3.2
- new net N$20: JP1.3, JP3.3
- new net N$21: JP1.4, JP3.4
- new net N$9: CAA.1, JP5.4
- new net VAIN: ICB.R, ICB.V+, JP5.3
- new net VBIN: ICA.R, ICA.V+, JP6.3
- net GND: now also CA.1, CAN.1, CB.1, CBN.1, ICA.GND, ICB.GND, JP5.1, JP6.1, PWR.2, RN1C.2, RN1D.2, X1.GND; no longer J-FEMALE.3
- net N$1: now also J-FEMALE.1, JP4.1; no longer J-FEMALE.4
- net N$12: now also RN1B.1; no longer RZ.1
- net N$2: now also JP4.2; no longer JP1.1
- net N$4: now also J-FEMALE.3, JP4.3; no longer X1.GND
- net N$6: now also J-FEMALE.4, JP4.4; no longer J-FEMALE.1
- net N$7: now also RN1B.2; no longer RZ.2
- net N$8: now also RN1A.1; no longer RC1.1
- net VBUS: now also RN1A.2; no longer RC1.2
- net VCC: now also JP5.2, JP6.2
- net VDD: now also PWR.1
Other:
- moved on the sheet: CAN, ICA, ICB, JP1, JP3, JP4, RA, RB

Commit message: update
Parts:
- removed JP2: (no value), pinhead:PINHD-1X18
Connections:
- net N$18: now also JP3.4; no longer JP3.1
- net N$19: now also JP1.3, JP3.1; no longer JP1.2, JP3.2
- net N$20: now also JP1.2; no longer JP1.3
- net N$21: now also JP3.2; no longer JP3.4
Other:
- moved on the sheet: JP1, JP3
Changed lines of the file:
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@@
 <part name="IC4" library="adafruit" deviceset="MCP1700" device="SOT89" value="MCP1700-33"/>
 <part name="BAT1" library="SparkFunNew" deviceset="BATTERY" device="BATTCOM_20MM_PTH_SMT" value="LIR2032"/>
-<part name="JP2" library="pinhead" deviceset="PINHD-1X18" device=""/>
 <part name="U$1" library="adafruit" deviceset="BUZZER" device=""/>
 <part name="RA" library="SparkFun-Connectors" deviceset="M02" device="PTH"/>
@@
 <instance part="CA" gate="G$1" x="105.41" y="92.71" rot="R270"/>
 <instance part="CB" gate="G$1" x="198.12" y="97.79" rot="R270"/>
-<instance part="JP1" gate="A" x="-34.29" y="83.82"/>
+<instance part="JP1" gate="A" x="-25.4" y="83.82"/>
 <instance part="X1" gate="G$1" x="-167.64" y="21.59" rot="R180"/>
 <instance part="GND5" gate="1" x="-87.63" y="-6.35" rot="MR0"/>
@@
 <attribute name="VALUE" x="-109.22" y="-2.032" size="1.778" layer="96"/>
 </instance>
-<instance part="JP2" gate="A" x="-116.84" y="66.04"/>
 <instance part="U$1" gate="G$1" x="-13.97" y="19.05" rot="R270"/>
 <instance part="RA" gate="G$1" x="120.65" y="92.71" rot="R270"/>
 <instance part="RB" gate="G$1" x="215.9" y="97.79" rot="R270"/>
 <instance part="PWR" gate="G$1" x="-12.7" y="55.88"/>
-<instance part="JP3" gate="A" x="-49.53" y="83.82"/>
+<instance part="JP3" gate="A" x="-57.15" y="82.55"/>
 <instance part="JP4" gate="A" x="10.16" y="100.33"/>
 <instance part="BZ" gate="G$1" x="-13.97" y="41.91" rot="R90"/>
@@
 <pinref part="BAT1" gate="G$1" pin="-"/>
 <wire x1="-104.14" y1="0.508" x2="-104.14" y2="-3.81" width="0.1524" layer="91"/>
+<junction x="-104.14" y="-3.81"/>
 </segment>
 <segment>
@@
 <wire x1="182.88" y1="60.96" x2="182.88" y2="66.04" width="0.1524" layer="91"/>
 <wire x1="193.04" y1="60.96" x2="182.88" y2="60.96" width="0.1524" layer="91"/>
+<junction x="182.88" y="60.96"/>
 </segment>
 <segment>
@@
 <pinref part="BAT1" gate="G$1" pin="+"/>
 <wire x1="-104.14" y1="10.668" x2="-104.14" y2="19.05" width="0.1524" layer="91"/>
+<junction x="-104.14" y="19.05"/>
 </segment>
 <segment>
@@
 <pinref part="RV1" gate="G$1" pin="2"/>
 <wire x1="146.05" y1="36.83" x2="158.75" y2="36.83" width="0.1524" layer="91"/>
+<junction x="135.89" y="36.83"/>
 </segment>
 </net>
@@
 <pinref part="JP6" gate="A" pin="5"/>
 <pinref part="RV2" gate="G$1" pin="2"/>
+<junction x="228.6" y="39.37"/>
 </segment>
 </net>
@@
 </segment>
 </net>
+<net name="N$19" class="0">
+<segment>
+<pinref part="JP1" gate="A" pin="3"/>
+<wire x1="-27.94" y1="83.82" x2="-45.72" y2="83.82" width="0.1524" layer="91"/>
+<wire x1="-45.72" y1="83.82" x2="-45.72" y2="87.63" width="0.1524" layer="91"/>
+<pinref part="JP3" gate="A" pin="1"/>
+<wire x1="-45.72" y1="87.63" x2="-59.69" y2="87.63" width="0.1524" layer="91"/>
+</segment>
+</net>
 <net name="N$18" class="0">
 <segment>
-<pinref part="JP3" gate="A" pin="1"/>
 <pinref part="JP1" gate="A" pin="1"/>
-<wire x1="-52.07" y1="88.9" x2="-36.83" y2="88.9" width="0.1524" layer="91"/>
-</segment>
-</net>
-<net name="N$19" class="0">
-<segment>
+<wire x1="-27.94" y1="88.9" x2="-41.91" y2="88.9" width="0.1524" layer="91"/>
+<wire x1="-41.91" y1="88.9" x2="-41.91" y2="80.01" width="0.1524" layer="91"/>
+<pinref part="JP3" gate="A" pin="4"/>
+<wire x1="-41.91" y1="80.01" x2="-59.69" y2="80.01" width="0.1524" layer="91"/>
+</segment>
+</net>
+<net name="N$20" class="0">
+<segment>
+<pinref part="JP1" gate="A" pin="2"/>
+<wire x1="-27.94" y1="86.36" x2="-44.45" y2="86.36" width="0.1524" layer="91"/>
+<wire x1="-44.45" y1="86.36" x2="-44.45" y2="82.55" width="0.1524" layer="91"/>
+<pinref part="JP3" gate="A" pin="3"/>
+<wire x1="-44.45" y1="82.55" x2="-59.69" y2="82.55" width="0.1524" layer="91"/>
+</segment>
+</net>
+<net name="N$21" class="0">
+<segment>
+<pinref part="JP1" gate="A" pin="4"/>
+<wire x1="-27.94" y1="81.28" x2="-39.37" y2="81.28" width="0.1524" layer="91"/>
+<wire x1="-39.37" y1="81.28" x2="-39.37" y2="85.09" width="0.1524" layer="91"/>
 <pinref part="JP3" gate="A" pin="2"/>
-<pinref part="JP1" gate="A" pin="2"/>
-<wire x1="-52.07" y1="86.36" x2="-36.83" y2="86.36" width="0.1524" layer="91"/>
-</segment>
-</net>
-<net name="N$20" class="0">
-<segment>
-<pinref part="JP3" gate="A" pin="3"/>
-<pinref part="JP1" gate="A" pin="3"/>
-<wire x1="-52.07" y1="83.82" x2="-36.83" y2="83.82" width="0.1524" layer="91"/>
-</segment>
-</net>
-<net name="N$21" class="0">
-<segment>
-<pinref part="JP3" gate="A" pin="4"/>
-<pinref part="JP1" gate="A" pin="4"/>
-<wire x1="-52.07" y1="81.28" x2="-36.83" y2="81.28" width="0.1524" layer="91"/>
-</segment>
-</net>
+<wire x1="-39.37" y1="85.09" x2="-59.69" y2="85.09" width="0.1524" layer="91"/>
+</segment>
+</net>

Commit message: update
Other:
- moved on the sheet: CA, CAA, CAN, CB, CBA, CBN, ICA, ICB, JP5, JP6, RA, RB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
