File: coqui-v1.0.sch (EAGLE design)
At the start: 32 parts, among them IC1 OPAMP-DUALU, IC3 MCP73831, IC4 MCP1700-33, J1 AYZ0202, X1 USBSMD

Commit message: update
Parts:
- removed CA1, RV1, RV2: (no value), pinhead:PINHD-1X1
- removed SV1, SV2: (no value), con-lstb:MA07-1
- added CB, RVA, RVB: M02PTH, SparkFun-Connectors:M02PTH
- added JP2, JP5: (no value), pinhead:PINHD-1X5
- CA: value (none) -> M02PTH; device pinhead:PINHD-1X1 -> SparkFun-Connectors:M02PTH
Connections:
- removed net N$17: SV1.6
- removed net N$25: CA.1, SV1.4
- removed net N$26: SV2.6
- removed net N$27: CA1.1, SV2.4
- net AOUT: now also JP2.4; no longer SV1.5
- net BOUT: now also JP5.4; no longer SV2.5
- net GND: now also CA.1, CB.1, JP2.1, JP5.1, RVA.2, RVB.1; no longer SV1.1
- net N$11: now also CA.2
- net N$13: now also JP5.5; no longer SV2.7
- net N$16: now also CB.2
- net N$23: now also RVA.1, RVB.2; no longer RV1.1
- net N$9: now also JP2.5; no longer SV1.7
- net VAIN: now also JP2.3; no longer SV1.3
- net VBIN: now also JP5.3
- net VCC: now also JP2.2, JP5.2; no longer SV1.2
