File: coqui-v1.0-linear.brd (EAGLE design)
At the start: 52.5 x 50.1 mm, 34 parts, among them IC1 OPAMP-DUALU, IC3 MCP73831, IC4 MCP1700-33, J1 AYZ0202, X1 USBSMD

Commit message: update
Parts:
- removed JP6, JP7: (no value), pinhead:1X12
- moved JP1 3.18 mm to (38.4, 7.37)
- moved CAN 2.67 mm to (0.76, 30.2), turned to 90 degrees
- moved JP3 2.54 mm to (31.6, 8.76)
- moved BATT 1.78 mm to (3.05, 17.4)
- moved BZ 1.48 mm to (6.35, 11.3)
- moved CHG 1.31 mm to (41.3, 14.2)
- moved ICB 1.27 mm to (46.2, 40.4), turned to 45 degrees
- moved ICA 1.09 mm to (4.06, 39.8)
- moved IC1 1.05 mm to (24.5, 20.7)
- moved X1 0.99 mm to (45.1, 5.84)
- moved IC4 0.90 mm to (48.3, 15.5)
- moved PWR 0.64 mm to (46.9, 21.1)
- moved CBN 0.63 mm to (48.9, 33.1)
- moved J1 0.57 mm to (47.6, 27.1)
- moved U$1 0.57 mm to (5.21, 5.33)
Routing:
- net GND: track 0.00 -> 218.7 mm, vias 0 -> 2
- net VBUS: track 0.00 -> 80.1 mm
- net AOUT: track 0.00 -> 78.9 mm, vias 0 -> 2
- net BOUT: track 0.00 -> 74.9 mm, vias 0 -> 1
- net VBIN: track 0.00 -> 72.8 mm, vias 0 -> 1
- net N$11: track 0.00 -> 70.4 mm, vias 0 -> 1
- net N$23: track 0.00 -> 69.0 mm, vias 0 -> 1
- net N$15: track 0.00 -> 62.2 mm, vias 0 -> 2
- net N$16: track 0.00 -> 59.5 mm, vias 0 -> 1
- net VAIN: track 0.00 -> 57.7 mm, vias 0 -> 1
- net N$7: track 0.00 -> 56.7 mm, vias 0 -> 2
- net VBAT: track 0.00 -> 54.5 mm, vias 0 -> 3
- net N$14: track 0.00 -> 51.9 mm
- net N$12: track 0.00 -> 50.9 mm, vias 0 -> 2
- net VCC: track 0.00 -> 46.4 mm, vias 0 -> 1
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Other:
- outline, holes or cut-outs redrawn
- board text added: "audio-based"
- board text added: "sensor"
