File: coqui-v1.0-linear.sch (EAGLE design)
At the start: 34 parts, among them IC1 OPAMP-DUALU, IC3 MCP73831, IC4 MCP1700-33, J1 AYZ0202, X1 USBSMD

Commit message: update
Parts:
- removed JP6, JP7: (no value), pinhead:PINHD-1X12
Changed lines of the file:
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@@
 <part name="JP2" library="pinhead" deviceset="PINHD-1X5" device=""/>
 <part name="JP5" library="pinhead" deviceset="PINHD-1X5" device=""/>
-<part name="JP6" library="pinhead" deviceset="PINHD-1X12" device=""/>
-<part name="JP7" library="pinhead" deviceset="PINHD-1X12" device=""/>
 </parts>
 <sheets>
@@
 <instance part="JP2" gate="A" x="-307.34" y="54.61" rot="R180"/>
 <instance part="JP5" gate="A" x="-157.48" y="54.61" rot="R180"/>
-<instance part="JP6" gate="G$1" x="-207.01" y="-26.67"/>
-<instance part="JP7" gate="G$1" x="-186.69" y="-24.13"/>
 </instances>
 <busses>
