File: coqui-v1.0.brd (EAGLE design)
At the start: 48.1 x 49.3 mm, 30 parts, among them IC3 MCP73831, IC4 MCP1700-33, J1 AYZ0202, X1 USBSMD

Commit message: update
Parts:
- removed CA, CB: M02PTH, SparkFun-Connectors:1X02
- removed JP5, JP6: (no value), pinhead:1X05
- added CB1: 0.01uF, rcl:C0805@1
- added IC1, IC2: OPAMP-DUALU, SparkFun-AnalogIC:SO08
- added JP2, JP7: (no value), pinhead:1X07
- added RV3: 22K, adafruit2013:R0805
- added SV1: (no value), con-lstb:MA04-1
- CAA, CAN, CBA, CBN: device rcl:C0805 -> rcl:C0805@1
Connections:
- new net N$22: IC2.4, RV3.2, SV1.2
- new net N$23: IC2.3, RV1.1, SV1.3
- new net V+: IC1.8
- new net V-: IC1.4
- net AOUT: now also JP2.7; no longer JP5.5, RN1.3
- net BOUT: now also ICA.3, JP7.7, RV3.1; no longer JP6.5
- net GND: now also JP2.2, JP2.3, JP7.2, JP7.3, SV1.1, SV1.4; no longer CA.1, CB.1, JP5.1, JP6.1, RN1.6
- net N$10: now also IC2.1, IC2.2, IC2.8; no longer RV1.1
- net N$11: now also JP2.1; no longer CA.2
- net N$16: now also JP7.1; no longer CB.2
- net N$17: now also JP7.6; no longer JP6.4
- net N$9: now also JP2.6; no longer JP5.4
- net VAIN: now also JP2.5; no longer JP5.3
- net VBIN: now also JP7.5; no longer JP6.3
- net VCC: now also JP2.4, JP7.4; no longer JP5.2, JP6.2
Routing:
- net GND: track 220.8 -> 157.7 mm
- net VCC: track 52.4 -> 22.2 mm
- net N$11: track 108.5 -> 97.0 mm
- net N$10: track 7.68 -> 0.00 mm

Commit message: update
Parts:
- removed CB1: 0.01uF, rcl:C0805@1
- removed IC2: OPAMP-DUALU, SparkFun-AnalogIC:SO08
- removed JP2, JP7: (no value), pinhead:1X07
- removed RV3: 22K, adafruit2013:R0805
- added CA, CA1: (no value), pinhead:1X01
- added RN2: (no value), resistor-dil:EXB38V
- added SV2: (no value), con-lstb:MA07-1
- RV1, RV2: value 22K -> (none); device adafruit2013:R0805 -> pinhead:1X01
- SV1: device con-lstb:MA04-1 -> con-lstb:MA07-1
- moved RV2 100.7 mm to (-1.27, -80.8)
- moved RV1 73.6 mm to (-1.27, -54.2), turned to 0 degrees
- moved IC1 37.4 mm to (29.8, 16.9)
- moved SV1 8.47 mm to (6.35, -47.2)
- moved CBA 2.90 mm to (31.0, 23.4)
- moved CAA 2.68 mm to (27.8, 23.2)
- moved RN1 1.99 mm to (33.7, 28.6)
- moved CHG 1.31 mm to (33.9, 16.1)
Connections:
- removed net N$22: IC2.4, RV3.2, SV1.2
- removed net V+: IC1.8
- removed net V-: IC1.4
- new net N$24: CBA.1, IC1.6, IC1.7
- new net N$25: CA.1, SV1.4
- new net N$26: SV2.6
- new net N$27: CA1.1, SV2.4
- net AOUT: now also RN2.8, SV1.5; no longer JP2.7, RV1.2
- net BOUT: now also RN2.2, SV2.5; no longer JP7.7, RN1.4, RV2.2, RV3.1
- net GND: now also IC1.8; no longer JP2.2, JP2.3, JP7.2, JP7.3, RN1.5, SV1.4
- net N$10: now also IC1.1, IC1.2; no longer IC2.1, IC2.2, IC2.8
- net N$11: no longer JP2.1
- net N$13: now also SV2.7; no longer RV2.1
- net N$16: no longer JP7.1
- net N$17: now also SV1.6; no longer CBA.1, JP7.6
- net N$23: now also IC1.3, IC1.5, RN2.1, RN2.7; no longer IC2.3, SV1.3
- net N$9: now also SV1.7; no longer JP2.6
- net VAIN: now also SV1.3; no longer JP2.5
- net VBIN: no longer JP7.5
- net VCC: now also IC1.4, SV1.2; no longer JP2.4, JP7.4
Routing:
- net GND: track 157.7 -> 0.00 mm, vias 3 -> 0
- net N$11: track 97.0 -> 0.00 mm, vias 1 -> 0
- net N$16: track 91.2 -> 0.00 mm, vias 3 -> 0
- net AOUT: track 85.5 -> 0.00 mm, vias 4 -> 0
- net VBIN: track 65.7 -> 0.00 mm, vias 1 -> 0
- net N$12: track 60.7 -> 0.00 mm, vias 2 -> 0
- net N$15: track 57.3 -> 0.00 mm, vias 2 -> 0
- net BOUT: track 51.7 -> 0.00 mm, vias 1 -> 0
- net VAIN: track 46.0 -> 0.00 mm, vias 2 -> 0
- net N$14: track 43.5 -> 0.00 mm
- net VBAT: track 38.5 -> 0.00 mm
- net VBUS: track 38.2 -> 0.00 mm, vias 3 -> 0
- net VDD: track 35.6 -> 0.00 mm, vias 2 -> 0
- net N$9: track 30.3 -> 0.00 mm
- net N$5: track 30.0 -> 0.00 mm
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
Commit message: update
Parts:
- removed CA1, RV1, RV2: (no value), pinhead:1X01
- removed SV1, SV2: (no value), con-lstb:MA07-1
- added CB, RVA, RVB: M02PTH, SparkFun-Connectors:1X02
- added JP2, JP5: (no value), pinhead:1X05
- CA: value (none) -> M02PTH; device pinhead:1X01 -> SparkFun-Connectors:1X02
- moved CA 90.5 mm to (11.3, 30.5), turned to 90 degrees
- moved ICB 32.9 mm to (46.2, 40.4), turned to 45 degrees
- moved ICA 31.9 mm to (4.06, 39.8), turned to 135 degrees
- moved CBN 31.5 mm to (48.9, 33.1), turned to 0 degrees
- moved IC4 30.9 mm to (48.3, 15.5), turned to 0 degrees
- moved U$1 30.0 mm to (5.21, 5.33)
- moved CAN 28.1 mm to (0.76, 30.2), turned to 90 degrees
- moved IC3 24.1 mm to (35.2, 19.4), turned to 0 degrees
- moved RN1 21.7 mm to (16.6, 42.0), turned to 230 degrees
- moved BZ 17.5 mm to (6.35, 11.3), turned to 180 degrees
- moved X1 17.5 mm to (45.1, 5.84), turned to 270 degrees
- moved RN2 13.7 mm to (34.9, 24.5)
- moved J1 12.8 mm to (47.6, 27.1), turned to 180 degrees
- moved PWR 11.8 mm to (46.9, 21.1), turned to 0 degrees
- moved CAA 9.68 mm to (18.5, 20.4)
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Connections:
- removed net N$17: SV1.6
- removed net N$25: CA.1, SV1.4
- removed net N$26: SV2.6
- removed net N$27: CA1.1, SV2.4
- net AOUT: now also JP2.4; no longer SV1.5
- net BOUT: now also JP5.4; no longer SV2.5
- net GND: now also CA.1, CB.1, JP2.1, JP5.1, RVA.2, RVB.1; no longer SV1.1
- net N$11: now also CA.2
- net N$13: now also JP5.5; no longer SV2.7
- net N$16: now also CB.2
- net N$23: now also RVA.1, RVB.2; no longer RV1.1
- net N$9: now also JP2.5; no longer SV1.7
- net VAIN: now also JP2.3; no longer SV1.3
- net VBIN: now also JP5.3
- net VCC: now also JP2.2, JP5.2; no longer SV1.2
Routing:
- net GND: track 0.00 -> 218.7 mm, vias 0 -> 2
- net VBUS: track 0.00 -> 80.1 mm
- net AOUT: track 0.00 -> 78.9 mm, vias 0 -> 2
- net BOUT: track 0.00 -> 74.9 mm, vias 0 -> 1
- net VBIN: track 0.00 -> 72.8 mm, vias 0 -> 1
- net N$11: track 0.00 -> 70.4 mm, vias 0 -> 1
- net N$23: track 0.00 -> 69.0 mm, vias 0 -> 1
- net N$15: track 0.00 -> 62.2 mm, vias 0 -> 2
- net N$16: track 0.00 -> 59.5 mm, vias 0 -> 1
- net VAIN: track 0.00 -> 57.7 mm, vias 0 -> 1
- net N$7: track 0.00 -> 56.7 mm, vias 0 -> 2
- net VBAT: track 0.00 -> 54.5 mm, vias 0 -> 3
- net N$14: track 0.00 -> 51.9 mm
- net N$12: track 0.00 -> 50.9 mm, vias 0 -> 2
- net VCC: track 0.00 -> 46.4 mm, vias 0 -> 1
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Other:
- board size 48.1 x 49.3 mm -> 52.5 x 50.1 mm
- board text added: "COQUI"
- board text added: "audio-based"
- board text added: "sensor"
- board text added: "v1.0"
- board text removed: "COQUI V1.0"
- board text removed: "off"
