File: coqui-v1.0.brd (EAGLE design)
At the start: 52.5 x 50.1 mm, 32 parts, among them IC1 OPAMP-DUALU, IC3 MCP73831, IC4 MCP1700-33, J1 AYZ0202, X1 USBSMD

Commit message: update
Other:
- board size 52.5 x 50.1 mm -> 52.7 x 50.2 mm
- board text removed: "audio-based"
- board text removed: "sensor"
Changed lines of the file:
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@@
 <text x="33.782" y="15.621" size="1.27" layer="21">IC3</text>
 <text x="45.212" y="15.113" size="1.27" layer="21" rot="R90">IC4</text>
-<wire x1="-0.762" y1="2.286" x2="2.413" y2="-0.127" width="0" layer="20" curve="90"/>
+<wire x1="-1.016" y1="2.286" x2="2.413" y2="-0.127" width="0" layer="20" curve="90"/>
 <wire x1="2.413" y1="-0.127" x2="46.99" y2="-0.127" width="0" layer="20"/>
 <wire x1="46.99" y1="-0.127" x2="51.689" y2="3.556" width="0" layer="20" curve="90"/>
-<wire x1="-0.762" y1="2.286" x2="-0.762" y2="39.878" width="0" layer="20"/>
-<wire x1="-0.762" y1="39.878" x2="6.096" y2="44.958" width="0" layer="20" curve="-90"/>
+<wire x1="-1.016" y1="2.286" x2="-1.016" y2="39.878" width="0" layer="20"/>
+<wire x1="-1.016" y1="39.878" x2="6.096" y2="44.958" width="0" layer="20" curve="-90"/>
 <wire x1="51.562" y1="39.878" x2="51.689" y2="3.556" width="0" layer="20"/>
 <text x="13.462" y="24.765" size="1.27" layer="21">O</text>
@@
 <wire x1="42.799" y1="35.814" x2="41.91" y2="34.925" width="0.254" layer="21" curve="-90"/>
 <wire x1="41.91" y1="34.925" x2="40.894" y2="34.925" width="0.254" layer="21"/>
-<text x="7.366" y="38.608" size="1.778" layer="21" rot="R245">audio-based</text>
-<text x="7.62" y="33.274" size="1.778" layer="21" rot="R245">sensor</text>
 </plain>
 <attributes>
@@
 </element>
 <element name="CAN" library="rcl" package="C0805@1" value="0.01uF" x="0.762" y="30.226" smashed="yes" rot="R90">
-<attribute name="NAME" x="0.127" y="33.147" size="1.27" layer="25"/>
+<attribute name="NAME" x="0.127" y="27.686" size="1.27" layer="25" rot="R270"/>
 <attribute name="VALUE" x="3.302" y="28.956" size="1.27" layer="27" rot="R90"/>
 </element>
@@
 <element name="U$1" library="adafruit" package="SMT-8585-BUZZER" value="BUZZER" x="5.207" y="5.334"/>
 <element name="RA" library="SparkFun-Connectors" package="1X02" value="M02PTH" x="11.303" y="43.18" smashed="yes" rot="R90">
-<attribute name="NAME" x="14.627440625" y="43.741053125" size="1.27" layer="25" ratio="10" rot="R90"/>
+<attribute name="NAME" x="16.456946875" y="46.504440625" size="1.27" layer="25" ratio="10" rot="R180"/>
 <attribute name="VALUE" x="14.47800625" y="41.909996875" size="1.27" layer="27" rot="R90"/>
 </element>
 <element name="RB" library="SparkFun-Connectors" package="1X02" value="M02PTH" x="39.243" y="45.847" smashed="yes" rot="R270">
-<attribute name="NAME" x="41.48195625" y="45.76440625" size="1.27" layer="25" ratio="10" rot="R270"/>
+<attribute name="NAME" x="41.35759375" y="44.91095625" size="1.27" layer="25" ratio="10"/>
 <attribute name="VALUE" x="36.068" y="47.117" size="1.27" layer="27" rot="R270"/>
 </element>
@@
 <attribute name="MF" value="" x="16.637" y="42.037" size="1.778" layer="27" rot="R230" display="off"/>
 <attribute name="OC_FARNELL" value="unknown" x="16.637" y="42.037" size="1.778" layer="27" rot="R230" display="off"/>
-<attribute name="NAME" x="16.88725" y="44.811171875" size="1.27" layer="25" rot="R320"/>
+<attribute name="NAME" x="19.196828125" y="40.25525" size="1.27" layer="25" rot="R50"/>
 <attribute name="VALUE" x="15.95914375" y="45.1807" size="1.27" layer="27" rot="R230"/>
 </element>
 <element name="IC1" library="SparkFun-AnalogIC" package="SO08" value="OPAMP-DUALU" x="24.511" y="20.701" rot="R90"/>
-<element name="RN2" library="resistor-dil" package="EXB38V" value="" x="34.925" y="24.511">
+<element name="RN2" library="resistor-dil" package="EXB38V" value="" x="34.925" y="24.511" smashed="yes">
 <attribute name="OC_NEWARK" value="unknown" x="34.925" y="24.511" size="1.778" layer="27" display="off"/>
 <attribute name="MPN" value="" x="34.925" y="24.511" size="1.778" layer="27" display="off"/>
 <attribute name="MF" value="" x="34.925" y="24.511" size="1.778" layer="27" display="off"/>
 <attribute name="OC_FARNELL" value="unknown" x="34.925" y="24.511" size="1.778" layer="27" display="off"/>
+<attribute name="NAME" x="34.2225" y="25.908" size="1.27" layer="25"/>
+<attribute name="VALUE" x="32.9525" y="21.971" size="1.27" layer="27"/>
 </element>
 <element name="CA" library="SparkFun-Connectors" package="1X02" value="M02PTH" x="11.303" y="30.48" smashed="yes" rot="R90">
